File: kicad/main.kicad_pcb (KiCad board)
At the start: 2 copper layers, 112.8 x 83.2 mm, 43 parts

Commit message: (Maybe) finished PCB
Parts:
- removed the G*** at (64.3, -15.6)
- removed the REF** at (104.1, -2.54) (x2)
- removed S18, S19, S20, S21, S22, S23, S24, S25, S26, S27, S28, S29, S30, S31, S32, S33, S34: , PG1350
- added G***: LOGO, project:silk_pattern_r, F.Cu at (64.4, -15.6)
- added G***: LOGO, project:silk_pattern_l, F.Cu at (64.2, -15.6)
- added REF**: OSHW-Logo_7.5x8mm_SilkScreen, Symbol:OSHW-Logo_7.5x8mm_SilkScreen, F.Cu at (104.1, -1.56)
- added REF**: OSHW-Logo_7.5x8mm_SilkScreen, Symbol:OSHW-Logo_7.5x8mm_SilkScreen, B.Cu at (104.1, -1.56)
- moved S17 81.4 mm to (105.7, 15.3), turned to -10 degrees
- moved S16 54.8 mm to (86.4, 13.6), turned to 0 degrees
- moved S10 41.4 mm to (72.0, -8.50), turned to 0 degrees
- moved S11 41.4 mm to (72.0, -25.5)
- moved S14 37.4 mm to (90.0, -23.8), turned to 0 degrees
- moved S15 37.4 mm to (90.0, -40.8)
- moved S13 36.6 mm to (90.0, -6.80)
- moved S12 36.2 mm to (72.0, -42.5), turned to 0 degrees
- moved S8 26.0 mm to (54.0, -30.6), turned to 0 degrees
- moved S9 26.0 mm to (54.0, -47.6)
- moved S6 21.6 mm to (36.0, -45.9), turned to 0 degrees
- moved S4 18.7 mm to (36.0, -11.9), turned to 0 degrees
- moved S5 18.7 mm to (36.0, -28.9)
- moved S7 18.1 mm to (54.0, -13.6)
- moved S2 17.0 mm to (18.0, -17.0), turned to 0 degrees
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Connections:
- S1 pad 1: P6 -> P8
- S10 pad 1: P4 -> P15
- S11 pad 1: P0 -> P4
- S13 pad 1: P7 -> P6
- S14 pad 1: P7 -> P20
- S15 pad 1: P19 -> P1
- S16 pad 1: P19 -> P9
- S17 pad 1: P2 -> P10
- S2 pad 1: P6 -> P18
- S3 pad 1: P20 -> P3
- S4 pad 1: P20 -> P14
- S5 pad 1: P1 -> P5
- S6 pad 1: P1 -> P21
- S7 pad 1: P15 -> P7
- S8 pad 1: P15 -> P19
- S9 pad 1: P4 -> P2
Routing:
- net GND: track 0.00 -> 766.3 mm, vias 0 -> 3
- net P18: track 0.00 -> 107.6 mm, vias 0 -> 1
- net P21: track 0.00 -> 105.4 mm, vias 0 -> 1
- net P8: track 0.00 -> 100.7 mm, vias 0 -> 1
- net P14: track 0.00 -> 98.7 mm, vias 0 -> 1
- net P3: track 0.00 -> 97.4 mm, vias 0 -> 1
- net P5: track 0.00 -> 94.6 mm, vias 0 -> 3
- net P19: track 0.00 -> 85.6 mm, vias 0 -> 3
- net P2: track 0.00 -> 70.5 mm, vias 0 -> 1
- net P7: track 0.00 -> 56.7 mm, vias 0 -> 1
- net RST: track 0.00 -> 55.2 mm
- net P15: track 0.00 -> 53.8 mm, vias 0 -> 1
- net P0: track 0.00 -> 42.1 mm, vias 0 -> 1
- net RAW: track 0.00 -> 41.1 mm, vias 0 -> 1
- net P4: track 0.00 -> 40.1 mm, vias 0 -> 1
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